Commit message: commit

File: src/space_robots_gz/simulation/models/canadarm/urdf/Canadarm2_w_iss.urdf (robot description, URDF)
Before this commit: robot SSRMS_Canadarm2, 9 links, 8 joints
Links:
- removed link world
- added link ISS, mass 1000.0; collision mesh filename=package://simulation/models/canadarm/meshes/iss.stl scale=1.0 1.0 1.0; visual mesh filename=package://simulation/models/canadarm/meshes/iss.dae scale=1.0 1.0 1.0
- link B1: geometry collision mesh filename=package://simulation/models/canadarm/meshes/joint_v3_0.stl scale=1.0 1.0 1.0; visual mesh filename=package://simulation/models/canadarm/meshes/joint_v3_0.dae scale=1.0 1.0 1.0
- link B2: geometry collision mesh filename=package://simulation/models/canadarm/meshes/joint_v3_0.stl scale=1.0 1.0 1.0; visual mesh filename=package://simulation/models/canadarm/meshes/joint_v3_0.dae scale=1.0 1.0 1.0
- link B3: geometry collision mesh filename=package://simulation/models/canadarm/meshes/joint_v3_0.stl scale=1.0 1.0 1.0; collision mesh filename=package://simulation/models/canadarm/meshes/joint_v3_0.stl scale=1.0 1.0 1.0
- link B4: geometry collision mesh filename=package://simulation/models/canadarm/meshes/joint_v3_0.stl scale=1.0 1.0 1.0; collision mesh filename=package://simulation/models/canadarm/meshes/link_joint_v2_1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 scale=1.0 1.0 1.0
- link B5: geometry collision mesh filename=package://simulation/models/canadarm/meshes/joint_v3_0.stl scale=1.0 1.0 1.0; visual mesh filename=package://simulation/models/canadarm/meshes/joint_v3_0.dae scale=1.0 1.0 1.0
- link B6: geometry collision mesh filename=package://simulation/models/canadarm/meshes/joint_v3_0.stl scale=1.0 1.0 1.0; visual mesh filename=package://simulation/models/canadarm/meshes/joint_v3_0.dae scale=1.0 1.0 1.0
- link Base_SSRMS: geometry collision mesh filename=package://simulation/models/canadarm/meshes/ee.stl scale=1.0 1.0 1.0; visual mesh filename=package://simulation/models/canadarm/meshes/ee.dae scale=1.0 1.0 1.0
- link EE_SSRMS: geometry collision mesh filename=package://simulation/models/canadarm/meshes/ee.stl scale=1.0 1.0 1.0; visual mesh filename=package://simulation/models/canadarm/meshes/ee.dae scale=1.0 1.0 1.0
Joints:
- removed joint world_joint
- added joint ISS_joint: type fixed, parent ISS, child Base_SSRMS, origin xyz=0 0 3.6 rpy=3.1416 0 0

File: src/space_robots_gz/simulation/models/canadarm/urdf/SSRMS_Canadarm2_w_iss.gazebo.xacro (robot description, xacro)
@@ -55,6 +55,4 @@
       <parameters>$(find canadarm)/config/canadarm_control.yaml</parameters>
       </plugin>
-      <!-- Base Link State Publisher-->
-      <plugin filename="libcanadarm_gz_plugin.so" name="canadarm_gz_plugin"></plugin>
   </gazebo>
   <!-- Colors -->
