Commit message: commit

File: src/space_robots_gz/simulation/models/canadarm/urdf/floating_canadaram.urdf.xacro (robot description, xacro)
@@ -26,5 +26,5 @@
     <origin rpy="0 0 0" xyz="0.0 0 -0.0"/>
     <axis xyz="1 0 0"/>
-    <limit lower="-10000.0" upper="10000.0" effort="5.0" velocity="5.0"/>
+    <limit lower="-10000.0" upper="10000.0" effort="1000.0" velocity="5.0"/>
   </joint>
   <link name="v_y_link">
@@ -40,5 +40,5 @@
     <origin rpy="0 0 0" xyz="0.0 0 -0.0"/>
     <axis xyz="0 1 0"/>
-    <limit lower="-10000.0" upper="10000.0" effort="5.0" velocity="5.0"/>
+    <limit lower="-10000.0" upper="10000.0" effort="1000.0" velocity="5.0"/>
   </joint>
   <link name="v_z_link">
@@ -54,5 +54,5 @@
     <origin rpy="0 0 0" xyz="0.0 0 -0.0"/>
     <axis xyz="0 0 1"/>
-    <limit lower="-10000.0" upper="10000.0" effort="5.0" velocity="5.0"/>
+    <limit lower="-10000.0" upper="10000.0" effort="1000.0" velocity="5.0"/>
   </joint>
     <link name="v_r_link">
@@ -68,5 +68,5 @@
     <origin rpy="0 0 0" xyz="0.0 0 -0.0"/>
     <axis xyz="1 0 0"/>
-    <limit lower="-6.28" upper="6.28" effort="5.0" velocity="5.0"/>
+    <limit lower="-6.28" upper="6.28" effort="1000.0" velocity="5.0"/>
   </joint>
     <link name="v_p_link">
@@ -82,5 +82,5 @@
     <origin rpy="0 0 0" xyz="0.0 0 -0.0"/>
     <axis xyz="0 1 0"/>
-    <limit lower="-6.28" upper="6.28" effort="5.0" velocity="5.0"/>
+    <limit lower="-6.28" upper="6.28" effort="1000.0" velocity="5.0"/>
   </joint>
     <link name="v_yaw_link">
@@ -96,5 +96,5 @@
     <origin rpy="0 0 0" xyz="0.0 0 -0.0"/>
     <axis xyz="0 0 1"/>
-    <limit lower="-6.28" upper="6.28" effort="5.0" velocity="5.0"/>
+    <limit lower="-6.28" upper="6.28" effort="1000.0" velocity="5.0"/>
   </joint>
   <link name="ISS">

File: src/space_robots_gz/simulation/models/canadarm/urdf/floating_canadarm.gazebo.xacro (robot description, xacro)
@@ -90,5 +90,5 @@
       <robot_param>robot_description</robot_param>
       <robot_param_node>robot_state_publisher</robot_param_node>
-      <parameters>$(find canadarm)/config/floating_canadaram_control.yaml</parameters>
+      <parameters>$(find canadarm)/config/floating_canadarm_control.yaml</parameters>
       </plugin>
   </gazebo>

File: src/space_robots_gz/simulation/models/franka/urdf/franka.gazebo.xacro (robot description, xacro)
@@ -4,5 +4,5 @@
   <ros2_control name="FrankaSystem" type="system">
       <hardware>
-          <plugin>ign_ros2_control/FrankaSystem</plugin>
+          <plugin>ign_ros2_control/IgnitionSystem</plugin>
       </hardware>
       <joint name="panda_joint1">

Commit message: commit

File: src/space_robots_gz/simulation/models/canadarm/urdf/floating_canadaram.urdf.xacro (robot description, xacro)
@@ -24,5 +24,5 @@
     <parent link="v_x_link"/>
     <child link="v_y_link"/>
-    <origin rpy="0 0 0" xyz="0.0 0 -0.0"/>
+    <origin rpy="0 0 0" xyz="0 0 0"/>
     <axis xyz="1 0 0"/>
     <limit lower="-10000.0" upper="10000.0" effort="1000.0" velocity="5.0"/>
@@ -38,5 +38,5 @@
     <parent link="v_y_link"/>
     <child link="v_z_link"/>
-    <origin rpy="0 0 0" xyz="0.0 0 -0.0"/>
+    <origin rpy="0 0 0" xyz="0 0 0"/>
     <axis xyz="0 1 0"/>
     <limit lower="-10000.0" upper="10000.0" effort="1000.0" velocity="5.0"/>
@@ -56,5 +56,5 @@
     <limit lower="-10000.0" upper="10000.0" effort="1000.0" velocity="5.0"/>
   </joint>
-    <link name="v_r_link">
+  <link name="v_r_link">
     <inertial>
       <mass value="0.00001"/>
@@ -70,5 +70,5 @@
     <limit lower="-6.28" upper="6.28" effort="1000.0" velocity="5.0"/>
   </joint>
-    <link name="v_p_link">
+  <link name="v_p_link">
     <inertial>
       <mass value="0.00001"/>
