Commit message: commit

File: src/space_robots_gz/simulation/models/canadarm/urdf/floating_canadarm_camera.gazebo.xacro (robot description, xacro)
@@ -98,11 +98,45 @@
         <update_frequency>10</update_frequency>
       </plugin>
+        <plugin filename="ignition-gazebo-sensors-system" name="ignition::gazebo::systems::Sensors">
+          <render_engine>ogre2</render_engine>
+      </plugin>
+  </gazebo>
+  <gazebo reference="camera_link">
+      <sensor type="camera" name="camera_sensor">
+          <visualize>1</visualize>
+          <update_rate>10.0</update_rate>
+          <camera>
+              <pose>1.0 0 0 0 0 -1.57</pose>
+              <horizontal_fov>1.3962634</horizontal_fov>
+              <image>
+                  <width>800</width>
+                  <height>800</height>
+                  <format>R8G8B8</format>
+              </image>
+              <clip>
+              <near>0.01</near>
+              <far>100</far>
+              </clip>
+              <noise>
+              <type>gaussian</type>
+              <stddev>0.007</stddev>
+              </noise>
+          </camera>
+          <always_on>1</always_on>
+          <topic>/SSRMS_camera/image_raw</topic>
+      </sensor>
   </gazebo>
   <!-- Colors -->
-  <material name="White">
-    <color rgba="1.0 1.0 1.0 1.0"/>
+  <material name="white">
+    <color rgba="1 1 1 1"/>
+  </material>
+  <material name="blue">
+    <color rgba="0 0 1 1"/>
+  </material>
+  <material name="red">
+    <color rgba="1 0 0 1"/>
   </material>
   <material name="green">
-    <color rgba="0 0.8 0 1"/>
+    <color rgba="0 1 0 1"/>
   </material>
   </xacro:macro>

File: src/space_robots_gz/simulation/models/ets_vii/urdf/ets_vii.gazebo.xacro (robot description, xacro)
@@ -6,4 +6,10 @@
           <plugin>ign_ros2_control/IgnitionSystem</plugin>
       </hardware>
+      <joint name="docking_interface_joint">
+          <command_interface name="${command_interface}"/>
+          <state_interface name="position"/>
+          <state_interface name="velocity"/>
+          <state_interface name="effort"/>
+      </joint>
       <joint name="joint1">
           <command_interface name="${command_interface}"/>
@@ -44,12 +50,25 @@
   </ros2_control>
   <gazebo>
-      <plugin filename="ignition-gazebo-pose-publisher-system" name="ignition::gazebo::systems::PosePublisher">
-        <publish_link_pose>true</publish_link_pose>
-        <publish_model_pose>true</publish_model_pose>
-        <publish_nested_model_pose>true</publish_nested_model_pose>
-        <use_pose_vector_msg>false</use_pose_vector_msg>
-        <update_frequency>10</update_frequency>
-      </plugin>
+    <plugin filename="ignition-gazebo-pose-publisher-system" name="ignition::gazebo::systems::PosePublisher">
+      <publish_link_pose>true</publish_link_pose>
+      <publish_model_pose>true</publish_model_pose>
+      <publish_nested_model_pose>true</publish_nested_model_pose>
+      <use_pose_vector_msg>false</use_pose_vector_msg>
+      <update_frequency>10</update_frequency>
+    </plugin>
   </gazebo>
+  <gazebo reference="docking_interface">
+    <material>Gazebo/White</material>
+  </gazebo>
+  <!-- Colors -->
+  <material name="white">
+    <color rgba="1 1 1 1"/>
+  </material>
+  <material name="blue">
+    <color rgba="0 0 1 1"/>
+  </material>
+  <material name="red">
+    <color rgba="1 0 0 1"/>
+  </material>
   </xacro:macro>
 </robot>

File: src/space_robots_gz/simulation/models/ets_vii/urdf/ets_vii.urdf.xacro (robot description, xacro)
@@ -20,4 +20,27 @@
     </inertial>
   </link>
+  <link name="docking_interface">
+    <visual>
+      <origin rpy="0 0 0" xyz="0 0 0" />
+      <geometry>
+        <box size="0.65 0.65 0.03" />
+      </geometry>
+      <material name="white"/>
+    </visual>
+    <collision>
+      <geometry>
+        <box size="0.65 0.65 0.03" />
+      </geometry>
+    </collision>
+    <inertial>
+      <mass value="0.01"/>
+      <inertia ixx="1.22" ixy="-0.0731" ixz="0.0007" iyy="0.513" iyz="0.113" izz="1.33"/>
+    </inertial>
+  </link>
+  <joint name="docking_interface_joint" type="fixed">
+    <parent link="base_link" />
+    <child link="docking_interface" />
+    <origin xyz="0.0 0 -1.0" rpy="0 0 0" />
+  </joint>
   <link name="link_1">
     <visual>

Commit message: commit

File: src/space_robots_gz/simulation/models/canadarm/urdf/floating_canadarm_camera.gazebo.xacro (robot description, xacro)
@@ -124,5 +124,31 @@
           </camera>
           <always_on>1</always_on>
-          <topic>/SSRMS_camera/image_raw</topic>
+          <topic>/SSRMS_camera/ee/image_raw</topic>
+      </sensor>
+  </gazebo>
+  <gazebo reference="base_camera_link">
+      <sensor type="camera" name="camera_sensor">
+          <visualize>1</visualize>
+          <update_rate>10.0</update_rate>
+          <camera>
+              <pose>1.0 0 0 0 0 -1.57</pose>
+              <!-- <horizontal_fov>1.3962634</horizontal_fov> -->
+              <horizontal_fov>1.7</horizontal_fov>
+              <image>
+                  <width>800</width>
+                  <height>800</height>
+                  <format>R8G8B8</format>
+              </image>
+              <clip>
+              <near>0.01</near>
+              <far>100</far>
+              </clip>
+              <noise>
+              <type>gaussian</type>
+              <stddev>0.007</stddev>
+              </noise>
+          </camera>
+          <always_on>1</always_on>
+          <topic>/SSRMS_camera/base/image_raw</topic>
       </sensor>
   </gazebo>

File: src/space_robots_gz/simulation/models/canadarm/urdf/floating_canadarm_camera.urdf.xacro (robot description, xacro)
@@ -414,3 +414,22 @@
     </visual>
 	</link>
+  <joint name="base_camera_joint" type="fixed">
+    <parent link="B1"/>
+    <child link="base_camera_link"/>
+    <origin xyz="-0.292 -0.003 -1.15" rpy="0 ${PI/2} 0"/>
+  </joint>
+  <link name="base_camera_link">
+    <inertial>
+      <origin xyz="0 0 0" rpy="0 0 0"/>
+      <mass value="0.001" />
+      <inertia ixx="9.1875e-09" ixy="0.0" ixz="0.0" iyy="9.1875e-09" iyz="0.0" izz="1.378125e-08"/>
+    </inertial>
+		<visual>
+      <origin rpy="0.0 0 0" xyz="0 0 0"/>
+      <geometry>
+        <box size="0.0005 0.0005 0.0005"/>
+      </geometry>
+      <material name="green"/>
+    </visual>
+	</link>
 </robot>
