Commit message: commit

File: src/space_robots_gz/simulation/models/canadarm/urdf/SSRMS_Canadarm2_w_iss.gazebo.xacro (robot description, xacro)
@@ -55,4 +55,6 @@
       <parameters>$(find canadarm)/config/canadarm_control.yaml</parameters>
       </plugin>
+      <!-- Base Link State Publisher-->
+      <plugin filename="libcanadarm_gz_plugin.so" name="canadarm_gz_plugin"></plugin>
   </gazebo>
   <!-- Colors -->

File: src/space_robots_gz/simulation/models/canadarm/urdf/SSRMS_Canadarm2_w_iss.urdf (robot description, URDF)
Before this commit: robot SSRMS_Canadarm2, 9 links, 8 joints
Links:
- removed link world
- added link ISS, mass 1000.0; collision mesh filename=package://simulation/models/canadarm/meshes/iss.stl scale=1.0 1.0 1.0; visual mesh filename=package://simulation/models/canadarm/meshes/iss.dae scale=1.0 1.0 1.0
- link B1: geometry collision mesh filename=package://simulation/models/canadarm/meshes/joint_v3_0.stl scale=1.0 1.0 1.0; visual mesh filename=package://simulation/models/canadarm/meshes/joint_v3_0.dae scale=1.0 1.0 1.0
- link B2: geometry collision mesh filename=package://simulation/models/canadarm/meshes/joint_v3_0.stl scale=1.0 1.0 1.0; visual mesh filename=package://simulation/models/canadarm/meshes/joint_v3_0.dae scale=1.0 1.0 1.0
- link B3: geometry collision mesh filename=package://simulation/models/canadarm/meshes/joint_v3_0.stl scale=1.0 1.0 1.0; collision mesh filename=package://simulation/models/canadarm/meshes/joint_v3_0.stl scale=1.0 1.0 1.0
- link B4: geometry collision mesh filename=package://simulation/models/canadarm/meshes/joint_v3_0.stl scale=1.0 1.0 1.0; collision mesh filename=package://simulation/models/canadarm/meshes/link_joint_v2_1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 scale=1.0 1.0 1.0
- link B5: geometry collision mesh filename=package://simulation/models/canadarm/meshes/joint_v3_0.stl scale=1.0 1.0 1.0; visual mesh filename=package://simulation/models/canadarm/meshes/joint_v3_0.dae scale=1.0 1.0 1.0
- link B6: geometry collision mesh filename=package://simulation/models/canadarm/meshes/joint_v3_0.stl scale=1.0 1.0 1.0; visual mesh filename=package://simulation/models/canadarm/meshes/joint_v3_0.dae scale=1.0 1.0 1.0
- link Base_SSRMS: geometry collision mesh filename=package://simulation/models/canadarm/meshes/ee.stl scale=1.0 1.0 1.0; visual mesh filename=package://simulation/models/canadarm/meshes/ee.dae scale=1.0 1.0 1.0
- link EE_SSRMS: geometry collision mesh filename=package://simulation/models/canadarm/meshes/ee.stl scale=1.0 1.0 1.0; visual mesh filename=package://simulation/models/canadarm/meshes/ee.dae scale=1.0 1.0 1.0
Joints:
- removed joint world_joint
- added joint ISS_joint: type fixed, parent ISS, child Base_SSRMS, origin xyz=0 0 3.6 rpy=3.1416 0 0

Commit message: commit

File: src/space_robots_gz/simulation/models/canadarm/urdf/SSRMS_Canadarm2_w_iss.gazebo.xacro (robot description, xacro)
@@ -1,5 +1,5 @@
 <?xml version="1.0" ?>
 <robot xmlns:xacro="http://wiki.ros.org/xacro">
-  <xacro:macro name="ssrms_canadarm2_gazebo" params="command_interface:=effort">
+  <xacro:macro name="ssrms_canadarm2_gazebo" params="command_interface:=position">
   <ros2_control name="IgnitionSystem" type="system">
       <hardware>

File: src/space_robots_gz/simulation/models/ets_vii/urdf/ets_vii.urdf.xacro (robot description, xacro)
@@ -37,5 +37,5 @@
     </inertial>
   </link>
-  <joint name="joint1" type="revolute">
+  <joint name="joint1" type="fixed">
     <axis xyz="0 0 1"/>
     <limit effort="1000.0" lower="-3.0" upper="3.0" velocity="0.5"/>
@@ -61,5 +61,5 @@
     </inertial>
   </link>
-  <joint name="joint2" type="revolute">
+  <joint name="joint2" type="fixed">
     <axis xyz="1 0 0"/>
     <limit effort="1000.0" lower="-3.0" upper="3.0" velocity="0.5"/>
@@ -85,5 +85,5 @@
     </inertial>
   </link>
-  <joint name="joint3" type="revolute">
+  <joint name="joint3" type="fixed">
     <axis xyz="-1 0 0"/>
     <limit effort="1000.0" lower="-3.0" upper="3.0" velocity="0.5"/>
@@ -109,5 +109,5 @@
     </inertial>
   </link>
-   <joint name="joint4" type="revolute">
+   <joint name="joint4" type="fixed">
     <axis xyz="1 0 0"/>
     <limit effort="1000.0" lower="-3.0" upper="3.0" velocity="0.5"/>
@@ -133,5 +133,5 @@
     </inertial>
   </link>
-   <joint name="joint5" type="revolute">
+   <joint name="joint5" type="fixed">
     <axis xyz="0 0 1"/>
     <limit effort="1000.0" lower="-3.0" upper="3.0" velocity="0.5"/>
@@ -157,5 +157,5 @@
     </inertial>
   </link>
-  <joint name="joint6" type="revolute">
+  <joint name="joint6" type="fixed">
     <axis xyz="1 0 0"/>
     <limit effort="1000.0" lower="-3.0" upper="3.0" velocity="0.5"/>

Commit message: commit

File: src/space_robots_gz/simulation/models/canadarm/urdf/SSRMS_Canadarm2_w_iss.gazebo.xacro (robot description, xacro)
@@ -51,12 +51,81 @@
   <gazebo>
       <plugin filename="libign_ros2_control-system" name="ign_ros2_control::IgnitionROS2ControlPlugin">
-      <robot_param>robot_description</robot_param>
-      <robot_param_node>robot_state_publisher</robot_param_node>
-      <parameters>$(find canadarm)/config/canadarm_control.yaml</parameters>
+        <robot_param>robot_description</robot_param>
+        <robot_param_node>robot_state_publisher</robot_param_node>
+        <parameters>$(find canadarm)/config/canadarm_control.yaml</parameters>
+      </plugin>
+      <plugin filename="ignition-gazebo-pose-publisher-system" name="ignition::gazebo::systems::PosePublisher">
+        <publish_model_pose>true</publish_model_pose>
+        <publish_nested_model_pose>true</publish_nested_model_pose>
+        <use_pose_vector_msg>false</use_pose_vector_msg>
+        <update_frequency>10</update_frequency>
+      </plugin>
+        <plugin filename="ignition-gazebo-sensors-system" name="ignition::gazebo::systems::Sensors">
+          <render_engine>ogre2</render_engine>
       </plugin>
   </gazebo>
+  <gazebo reference="camera_link">
+      <sensor type="camera" name="camera_sensor">
+          <visualize>1</visualize>
+          <update_rate>10.0</update_rate>
+          <camera>
+              <pose>1.0 0 0 0 0 -1.57</pose>
+              <horizontal_fov>1.3962634</horizontal_fov>
+              <image>
+                  <width>800</width>
+                  <height>800</height>
+                  <format>R8G8B8</format>
+              </image>
+              <clip>
+              <near>0.01</near>
+              <far>100</far>
+              </clip>
+              <noise>
+              <type>gaussian</type>
+              <stddev>0.007</stddev>
+              </noise>
+          </camera>
+          <always_on>1</always_on>
+          <topic>/SSRMS_camera/ee/image_raw</topic>
+      </sensor>
+  </gazebo>
+  <gazebo reference="base_camera_link">
+      <sensor type="camera" name="camera_sensor">
+          <visualize>1</visualize>
+          <update_rate>10.0</update_rate>
+          <camera>
+              <pose>1.0 0 0 0 0 -1.57</pose>
+              <!-- <horizontal_fov>1.3962634</horizontal_fov> -->
+              <horizontal_fov>1.7</horizontal_fov>
+              <image>
+                  <width>800</width>
+                  <height>800</height>
+                  <format>R8G8B8</format>
+              </image>
+              <clip>
+              <near>0.01</near>
+              <far>100</far>
+              </clip>
+              <noise>
+              <type>gaussian</type>
+              <stddev>0.007</stddev>
+              </noise>
+          </camera>
+          <always_on>1</always_on>
+          <topic>/SSRMS_camera/base/image_raw</topic>
+      </sensor>
+  </gazebo>
   <!-- Colors -->
-  <material name="White">
-    <color rgba="1.0 1.0 1.0 1.0"/>
+  <material name="white">
+    <color rgba="1 1 1 1"/>
+  </material>
+  <material name="blue">
+    <color rgba="0 0 1 1"/>
+  </material>
+  <material name="red">
+    <color rgba="1 0 0 1"/>
+  </material>
+  <material name="green">
+    <color rgba="0 1 0 1"/>
   </material>
   </xacro:macro>

File: src/space_robots_gz/simulation/models/canadarm/urdf/SSRMS_Canadarm2_w_iss.urdf.xacro (robot description, xacro)
@@ -8,4 +8,5 @@
   <xacro:include filename="$(find simulation)/models/canadarm/urdf/SSRMS_Canadarm2_w_iss.gazebo.xacro" />
   <xacro:ssrms_canadarm2_gazebo command_interface="position" />
+  <xacro:property name="PI" value="3.1415926535897931"/>
   <link name="world" />
   <joint name="world_joint" type="fixed">
@@ -310,3 +311,41 @@
     </collision>
   </link>
+  <joint name="head_camera_joint" type="fixed">
+    <parent link="EE_SSRMS"/>
+    <child link="camera_link"/>
+    <origin xyz="-0.292 -0.003 -1.15" rpy="0 ${PI/2} 0"/>
+  </joint>
+  <link name="camera_link">
+    <inertial>
+      <origin xyz="0 0 0" rpy="0 0 0"/>
+      <mass value="0.001" />
+      <inertia ixx="9.1875e-09" ixy="0.0" ixz="0.0" iyy="9.1875e-09" iyz="0.0" izz="1.378125e-08"/>
+    </inertial>
+		<visual>
+      <origin rpy="0.0 0 0" xyz="0 0 0"/>
+      <geometry>
+        <box size="0.0005 0.0005 0.0005"/>
+      </geometry>
+      <material name="green"/>
+    </visual>
+	</link>
+  <joint name="base_camera_joint" type="fixed">
+    <parent link="B1"/>
+    <child link="base_camera_link"/>
+    <origin xyz="-0.292 -0.003 -1.15" rpy="0 ${PI/2} 0"/>
+  </joint>
+  <link name="base_camera_link">
+    <inertial>
+      <origin xyz="0 0 0" rpy="0 0 0"/>
+      <mass value="0.001" />
+      <inertia ixx="9.1875e-09" ixy="0.0" ixz="0.0" iyy="9.1875e-09" iyz="0.0" izz="1.378125e-08"/>
+    </inertial>
+		<visual>
+      <origin rpy="0.0 0 0" xyz="0 0 0"/>
+      <geometry>
+        <box size="0.0005 0.0005 0.0005"/>
+      </geometry>
+      <material name="green"/>
+    </visual>
+	</link>
 </robot>
