Commit message: commit

File: src/space_robots_gz/simulation/models/canadarm/urdf/SSRMS_Canadarm2_w_iss.urdf.xacro (robot description, xacro)
@@ -7,5 +7,11 @@
   <!-- Gazebo - ROS2 Control macro -->
   <xacro:include filename="$(find simulation)/models/canadarm/urdf/SSRMS_Canadarm2_w_iss.gazebo.xacro" />
-  <xacro:ssrms_canadarm2_gazebo command_interface="position" />
+  <xacro:ssrms_canadarm2_gazebo command_interface="effort" />
+  <link name="world" />
+  <joint name="world_joint" type="fixed">
+    <parent link="world"/>
+    <child link="ISS"/>
+    <origin rpy="0 0 0" xyz="0 0 0"/>
+  </joint>
   <link name="ISS">
     <inertial>

Commit message: commit

File: src/space_robots_gz/simulation/models/canadarm/urdf/SSRMS_Canadarm2_w_iss.urdf.xacro (robot description, xacro)
@@ -7,5 +7,5 @@
   <!-- Gazebo - ROS2 Control macro -->
   <xacro:include filename="$(find simulation)/models/canadarm/urdf/SSRMS_Canadarm2_w_iss.gazebo.xacro" />
-  <xacro:ssrms_canadarm2_gazebo command_interface="position" />
+  <xacro:ssrms_canadarm2_gazebo command_interface="effort" />
   <xacro:property name="PI" value="3.1415926535897931"/>
   <link name="world" />

File: src/space_robots_gz/simulation/models/canadarm/urdf/floating_canadarm.urdf.xacro (robot description, xacro)
@@ -7,5 +7,5 @@
   <!-- Gazebo - ROS2 Control macro -->
   <xacro:include filename="$(find simulation)/models/canadarm/urdf/floating_canadarm.gazebo.xacro" />
-  <xacro:floating_canadarm_gazebo command_interface="position" />
+  <xacro:floating_canadarm_gazebo command_interface="effort" />
   <link name="world" />
   <joint name="world_to_vx" type="fixed">

File: src/space_robots_gz/simulation/models/franka/urdf/franka.gazebo.xacro (robot description, xacro)
@@ -1,5 +1,5 @@
 <?xml version="1.0" ?>
 <robot xmlns:xacro="http://wiki.ros.org/xacro">
-  <xacro:macro name="franka_gazebo" params="command_interface:=position">
+  <xacro:macro name="franka_gazebo" params="command_interface:=effort">
   <ros2_control name="FrankaSystem" type="system">
       <hardware>

File: src/space_robots_gz/simulation/models/franka/urdf/franka.urdf.xacro (robot description, xacro)
@@ -6,5 +6,5 @@
 <robot name="panda" xmlns:xacro="http://www.ros.org/wiki/xacro">
   <xacro:include filename="$(find simulation)/models/franka/urdf/franka.gazebo.xacro" />
-  <xacro:franka_gazebo command_interface="position" />
+  <xacro:franka_gazebo command_interface="effort" />
   <link name='world'>
   </link>
