Commit message: commit

File: src/mppi_controller/mppi_controller/models/canadarm/urdf/Canadarm2_w_iss.urdf (robot description, URDF)
Before this commit: robot SSRMS_Canadarm2, 9 links, 8 joints
Links:
- link B1: geometry collision mesh filename=package://mppi_controller/models/canadarm/meshes/joint_v3_0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 scale=1.0 1.0 1.0; visual mesh filename=package://mppi_controller/models/canadarm/meshes/joint_v3_0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 scale=1.0 1.0 1.0
- link B2: geometry collision mesh filename=package://mppi_controller/models/canadarm/meshes/joint_v3_0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 scale=1.0 1.0 1.0; visual mesh filename=package://mppi_controller/models/canadarm/meshes/joint_v3_0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 scale=1.0 1.0 1.0
- link B3: geometry collision mesh filename=package://mppi_controller/models/canadarm/meshes/joint_v3_0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 scale=1.0 1.0 1.0; collision mesh filename=package://mppi_controller/models/canadarm/meshes/joint_v3_0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 scale=1.0 1.0 1.0
- link B4: geometry collision mesh filename=package://mppi_controller/models/canadarm/meshes/joint_v3_0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 scale=1.0 1.0 1.0; collision mesh filename=package://mppi_controller/models/canadarm/meshes/link_joint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 scale=1.0 1.0 1.0
- link B5: geometry collision mesh filename=package://mppi_controller/models/canadarm/meshes/joint_v3_0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 scale=1.0 1.0 1.0; visual mesh filename=package://mppi_controller/models/canadarm/meshes/joint_v3_0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 scale=1.0 1.0 1.0
- link B6: geometry collision mesh filename=package://mppi_controller/models/canadarm/meshes/joint_v3_0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 scale=1.0 1.0 1.0; visual mesh filename=package://mppi_controller/models/canadarm/meshes/joint_v3_0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 scale=1.0 1.0 1.0
- link Base_SSRMS: geometry collision mesh filename=package://mppi_controller/models/canadarm/meshes/ee.stl scale=1.0 1.0 1.0; visual mesh filename=package://mppi_controller/models/canadarm/meshes/ee.dae scale=1.0 1.0 1.0
- link EE_SSRMS: geometry collision mesh filename=package://mppi_controller/models/canadarm/meshes/ee.stl scale=1.0 1.0 1.0; visual mesh filename=package://mppi_controller/models/canadarm/meshes/ee.dae scale=1.0 1.0 1.0
- link ISS: geometry collision mesh filename=package://mppi_controller/models/canadarm/meshes/iss.stl scale=1.0 1.0 1.0; visual mesh filename=package://mppi_controller/models/canadarm/meshes/iss.dae scale=1.0 1.0 1.0

File: src/space_robots_gz/simulation/models/ets_vii/urdf/ets_vii.gazebo.xacro (robot description, xacro)
@@ -1,10 +1,10 @@
 <?xml version="1.0" ?>
 <robot xmlns:xacro="http://wiki.ros.org/xacro">
-  <xacro:macro name="ssrms_canadarm2_gazebo" params="command_interface:=effort">
+  <xacro:macro name="ets_vii_gazebo" params="command_interface:=effort">
   <ros2_control name="IgnitionSystem" type="system">
       <hardware>
           <plugin>ign_ros2_control/IgnitionSystem</plugin>
       </hardware>
-      <joint name="Base_Joint">
+      <joint name="joint1">
           <command_interface name="${command_interface}"/>
           <state_interface name="position"/>
@@ -12,5 +12,5 @@
           <state_interface name="effort"/>
       </joint>
-      <joint name="Shoulder_Roll">
+      <joint name="joint2">
           <command_interface name="${command_interface}"/>
           <state_interface name="position"/>
@@ -18,5 +18,5 @@
           <state_interface name="effort"/>
       </joint>
-      <joint name="Shoulder_Yaw">
+      <joint name="joint3">
           <command_interface name="${command_interface}"/>
           <state_interface name="position"/>
@@ -24,5 +24,5 @@
           <state_interface name="effort"/>
       </joint>
-      <joint name="Elbow_Pitch">
+      <joint name="joint4">
           <command_interface name="${command_interface}"/>
           <state_interface name="position"/>
@@ -30,5 +30,5 @@
           <state_interface name="effort"/>
       </joint>
-      <joint name="Wrist_Pitch">
+      <joint name="joint5">
           <command_interface name="${command_interface}"/>
           <state_interface name="position"/>
@@ -36,11 +36,5 @@
           <state_interface name="effort"/>
       </joint>
-      <joint name="Wrist_Yaw">
-          <command_interface name="${command_interface}"/>
-          <state_interface name="position"/>
-          <state_interface name="velocity"/>
-          <state_interface name="effort"/>
-      </joint>
-      <joint name="Wrist_Roll">
+      <joint name="joint6">
           <command_interface name="${command_interface}"/>
           <state_interface name="position"/>
@@ -49,15 +43,11 @@
       </joint>
   </ros2_control>
-  <gazebo>
+  <!-- <gazebo>
       <plugin filename="libign_ros2_control-system" name="ign_ros2_control::IgnitionROS2ControlPlugin">
-      <robot_param>robot_description</robot_param>
-      <robot_param_node>robot_state_publisher</robot_param_node>
-      <parameters>$(find canadarm)/config/canadarm_control_w_satellite.yaml</parameters>
+        <robot_param>ets_vii_robot_description</robot_param>
+        <robot_param_node>ets_vii_robot_state_publisher</robot_param_node>
+        <parameters>$(find canadarm)/config/canadarm_control_w_satellite.yaml</parameters>
       </plugin>
-  </gazebo>
-  <!-- Colors -->
-  <material name="White">
-    <color rgba="1.0 1.0 1.0 1.0"/>
-  </material>
+  </gazebo> -->
   </xacro:macro>
 </robot>

File: src/space_robots_gz/simulation/models/ets_vii/urdf/ets_vii.urdf.xacro (robot description, xacro)
@@ -1,5 +1,6 @@
 <?xml version="1.0"?>
 <robot name="ets_vii" xmlns:xacro="http://www.ros.org/wiki/xacro">
-  <xacro:property name="pi" value="3.14159265"/>
+  <xacro:include filename="$(find simulation)/models/ets_vii/urdf/ets_vii.gazebo.xacro" />
+  <xacro:ets_vii_gazebo command_interface="effort" />
   <link name="base_link">
     <visual>
@@ -129,5 +130,5 @@
     <inertial>
       <mass value="26.2"/>
-      <inertia ixx="0.57" ixy="0" ixz="-0.231" iyy="0.599" iyz="0" izz="0.129"/>
+      <inertia ixx="0.57" ixy="0" ixz="-0.231" iyy="0.599" iyz="0" izz="0.258"/>
     </inertial>
   </link>
@@ -156,5 +157,5 @@
     </inertial>
   </link>
-   <joint name="joint6" type="revolute">
+  <joint name="joint6" type="revolute">
     <axis xyz="1 0 0"/>
     <limit effort="1000.0" lower="-3.0" upper="3.0" velocity="0.5"/>
