Commit message: commit

File: src/mppi_solver/mppi_solver/models/ets_vii/ets_vii.urdf (robot description, URDF)
Before this commit: robot ets_vii, 8 links, 7 joints
Joints:
- joint joint1: origin xyz=-0.79 -0.29 1 rpy=0.0 0.0 ${0.5 * pi} -> xyz=-0.79 -0.29 1 rpy=0.0 0.0 1.5707963267948966
- joint joint3: origin xyz=-0.125 0 0.87 rpy=${0.5 * pi} 0.0 0.0 -> xyz=-0.125 0 0.87 rpy=1.5707963267948966 0.0 0.0
- joint joint4: origin xyz=-0.262 0 0.63 rpy=${-0.5 * pi} 0.0 0.0 -> xyz=-0.262 0 0.63 rpy=-1.5707963267948966 0.0 0.0
- joint joint5: origin xyz=0 0 0.277 rpy=0.0 0.0 ${-0.5 * pi} -> xyz=0 0 0.277 rpy=0.0 0.0 -1.5707963267948966
